Commit message: reactivated state action server in controller, added dummy link to youbot base for KDL

File: youbot_description/urdf/youbot_base/base.urdf.xacro (robot description, xacro)
@@ -32,4 +32,11 @@
 	<xacro:macro name="youbot_base" params="name">
 		<link name="${name}_footprint">
+    		</link>
+    		<joint name="${name}_footprint_fixer" type="fixed">
+      			<origin xyz="0 0 0" rpy="0 0 0" />
+      			<child link="${name}_footprint_inertia" />
+      			<parent link="${name}_footprint"/>
+    		</joint>
+		<link name="${name}_footprint_inertia">
       			<inertial>
         			<mass value="0.1" />
