Commit message: -

File: youbot_description/urdf/youbot_arm/arm_with_cam.urdf.xacro (robot description, xacro)
@@ -212,5 +212,5 @@
 		</link>
 		<joint name="cameramount" type="fixed">
-		  <origin xyz="-0.04 0 0" rpy="0 ${-M_PI/2.0} 0" />
+		  <origin xyz="-0.04 0 0" rpy="0 ${-M_PI/2.0} 0" /><!--<origin xyz="-0.04 0 0" rpy="${M_PI/2} 0 ${-M_PI/2.0}" />-->
 		  <parent link="${name}_link_5"/>
 		  <child link="camera" />
