Commit message: changing gazebo camera topic to /camera/image_rect

File: youbot_description/urdf/youbot_arm/arm_with_cam.gazebo.xacro (robot description, xacro)
@@ -45,5 +45,5 @@
 		      <alwaysOn>true</alwaysOn>
 		      <updateRate>30.0</updateRate>
-		      <cameraName>youbot/eye</cameraName>
+		      <cameraName>camera</cameraName>
 		      <imageTopicName>image_rect</imageTopicName>
 		      <cameraInfoTopicName>camera_info</cameraInfoTopicName>

File: youbot_description/urdf/youbot_arm/arm_with_cam.urdf.xacro (robot description, xacro)
@@ -212,5 +212,6 @@
 		</link>
 		<joint name="cameramount" type="fixed">
-		  <origin xyz="-0.04 0 0" rpy="0 ${-M_PI/2.0} 0" /><!--<origin xyz="-0.04 0 0" rpy="${M_PI/2} 0 ${-M_PI/2.0}" />-->
+		  <!-- camera pointing forward or sideways -->
+		  <!--<origin xyz="-0.04 0 0" rpy="0 ${-M_PI/2.0} 0" />--><origin xyz="-0.04 0 0" rpy="${M_PI/2} 0 ${-M_PI/2.0}" />
 		  <parent link="${name}_link_5"/>
 		  <child link="camera" />
